File: HMC799/circular3_HMC799.kicad_pcb (KiCad board)
At the start: 2 copper layers, 25 x 25 mm, 37 parts, among them J101 Conn_Coaxial, J102 Conn_01x03, U101 LT3042xMSE, U102 LT3094xMSE, U103 HMC799LP3E, U104 BUF602xDBV

Commit message: minor
Parts:
- J101: moved to B.Cu
- turned J101 to 315 degrees
Changed lines of the file:
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@@
-(kicad_pcb (version 20171130) (host pcbnew 5.1.5-52549c5~86~ubuntu18.04.1)
+(kicad_pcb (version 20171130) (host pcbnew 5.1.5-52549c5~86~ubuntu19.10.1)
   (general
     (thickness 1.6)
@@
     )
   )
-  (module Connector_Coaxial:MMCX_Molex_73415-1471_Vertical (layer F.Cu)
-    (at 146.25 93 45)
+  (module Connector_Coaxial:MMCX_Molex_73415-1471_Vertical (layer B.Cu)
+    (at 146.25 93 315)
     (descr http://www.molex.com/pdm_docs/sd/734151471_sd.pdf)
     (tags "Molex MMCX Coaxial Connector 50 ohms Female Jack Vertical THT")
-    (fp_text reference J101 (at 0 0 45) (layer F.SilkS) hide
-      (effects (font (size 0.5 0.5) (thickness 0.1)))
-    )
-    (fp_text value Conn_Coaxial (at 0 3.2 45) (layer F.Fab)
-      (effects (font (size 1 1) (thickness 0.15)))
-    )
-    (fp_line (start 0.62 1.87) (end -0.62 1.87) (layer F.SilkS) (width 0.12))
-    (fp_line (start 0.62 -1.87) (end -0.62 -1.87) (layer F.SilkS) (width 0.12))
-    (fp_line (start -1.87 0.62) (end -1.87 -0.62) (layer F.SilkS) (width 0.12))
-    (fp_line (start -2.39 2.39) (end -2.39 -2.39) (layer F.CrtYd) (width 0.05))
-    (fp_line (start 1.87 0.62) (end 1.87 -0.62) (layer F.SilkS) (width 0.12))
-    (fp_line (start -1.755 1.755) (end 1.755 1.755) (layer F.Fab) (width 0.1))
-    (fp_line (start -1.755 -1.755) (end 1.755 -1.755) (layer F.Fab) (width 0.1))
-    (fp_line (start 1.755 -1.755) (end 1.755 1.755) (layer F.Fab) (width 0.1))
-    (fp_line (start -1.755 -1.755) (end -1.755 1.755) (layer F.Fab) (width 0.1))
-    (fp_line (start 2.39 2.39) (end 2.39 -2.39) (layer F.CrtYd) (width 0.05))
-    (fp_line (start -2.39 -2.39) (end 2.39 -2.39) (layer F.CrtYd) (width 0.05))
-    (fp_line (start -2.39 2.39) (end 2.39 2.39) (layer F.CrtYd) (width 0.05))
-    (fp_text user %R (at 0 0 45) (layer F.Fab)
-      (effects (font (size 0.5 0.5) (thickness 0.1)))
-    )
-    (pad 2 thru_hole circle (at -1.27 1.27 45) (size 1.24 1.24) (drill 0.84) (layers *.Cu *.Mask)
-      (net 2 GND))
-    (pad 2 thru_hole circle (at 1.27 -1.27 45) (size 1.24 1.24) (drill 0.84) (layers *.Cu *.Mask)
-      (net 2 GND))
-    (pad 2 thru_hole circle (at 1.27 1.27 45) (size 1.24 1.24) (drill 0.84) (layers *.Cu *.Mask)
-      (net 2 GND))
-    (pad 2 thru_hole circle (at -1.27 -1.27 45) (size 1.24 1.24) (drill 0.84) (layers *.Cu *.Mask)
+    (fp_text reference J101 (at 0 0 315) (layer B.SilkS) hide
+      (effects (font (size 0.5 0.5) (thickness 0.1)) (justify mirror))
+    )
+    (fp_text value Conn_Coaxial (at 0 -3.2 315) (layer B.Fab)
+      (effects (font (size 1 1) (thickness 0.15)) (justify mirror))
+    )
+    (fp_line (start 0.62 -1.87) (end -0.62 -1.87) (layer B.SilkS) (width 0.12))
+    (fp_line (start 0.62 1.87) (end -0.62 1.87) (layer B.SilkS) (width 0.12))
+    (fp_line (start -1.87 -0.62) (end -1.87 0.62) (layer B.SilkS) (width 0.12))
+    (fp_line (start -2.39 -2.39) (end -2.39 2.39) (layer B.CrtYd) (width 0.05))
+    (fp_line (start 1.87 -0.62) (end 1.87 0.62) (layer B.SilkS) (width 0.12))
+    (fp_line (start -1.755 -1.755) (end 1.755 -1.755) (layer B.Fab) (width 0.1))
+    (fp_line (start -1.755 1.755) (end 1.755 1.755) (layer B.Fab) (width 0.1))
+    (fp_line (start 1.755 1.755) (end 1.755 -1.755) (layer B.Fab) (width 0.1))
+    (fp_line (start -1.755 1.755) (end -1.755 -1.755) (layer B.Fab) (width 0.1))
+    (fp_line (start 2.39 -2.39) (end 2.39 2.39) (layer B.CrtYd) (width 0.05))
+    (fp_line (start -2.39 2.39) (end 2.39 2.39) (layer B.CrtYd) (width 0.05))
+    (fp_line (start -2.39 -2.39) (end 2.39 -2.39) (layer B.CrtYd) (width 0.05))
+    (fp_text user %R (at 0 0 315) (layer B.Fab)
+      (effects (font (size 0.5 0.5) (thickness 0.1)) (justify mirror))
+    )
+    (pad 2 thru_hole circle (at -1.27 -1.27 315) (size 1.24 1.24) (drill 0.84) (layers *.Cu *.Mask)
+      (net 2 GND))
+    (pad 2 thru_hole circle (at 1.27 1.27 315) (size 1.24 1.24) (drill 0.84) (layers *.Cu *.Mask)
+      (net 2 GND))
+    (pad 2 thru_hole circle (at 1.27 -1.27 315) (size 1.24 1.24) (drill 0.84) (layers *.Cu *.Mask)
+      (net 2 GND))
+    (pad 2 thru_hole circle (at -1.27 1.27 315) (size 1.24 1.24) (drill 0.84) (layers *.Cu *.Mask)
       (net 2 GND) (zone_connect 1) (thermal_width 0.5))
-    (pad 1 thru_hole circle (at 0 0 45) (size 1.24 1.24) (drill 0.84) (layers *.Cu *.Mask)
+    (pad 1 thru_hole circle (at 0 0 315) (size 1.24 1.24) (drill 0.84) (layers *.Cu *.Mask)
       (net 9 "Net-(J101-Pad1)"))
     (model ${KISYS3DMOD}/Connector_Coaxial.3dshapes/MMCX_Molex_73415-1471_Vertical.wrl
@@
   (gr_line (start 150 150) (end 150 50) (layer Dwgs.User) (width 0.15))
   (gr_line (start 100 100) (end 200 100) (layer Dwgs.User) (width 0.15))
-  (via (at 139.9 100.5) (size 0.8) (drill 0.4) (layers F.Cu B.Cu) (net 2))
-  (via (at 139.9 102) (size 0.8) (drill 0.4) (layers F.Cu B.Cu) (net 2))
-  (via (at 140.2 99.2) (size 0.8) (drill 0.4) (layers F.Cu B.Cu) (net 2))
   (segment (start 150.02 102.7325) (end 150.0375 102.75) (width 0.35) (layer B.Cu) (net 1))
   (segment (start 150.02 101.27) (end 150.02 102.7325) (width 0.35) (layer B.Cu) (net 1))
   (segment (start 150 101.29) (end 150.02 101.27) (width 0.3) (layer B.Cu) (net 1))
   (segment (start 150 102.7125) (end 150 101.29) (width 0.3) (layer B.Cu) (net 1))
+  (via (at 139.9 100.5) (size 0.8) (drill 0.4) (layers F.Cu B.Cu) (net 2))
+  (via (at 139.9 102) (size 0.8) (drill 0.4) (layers F.Cu B.Cu) (net 2))
+  (via (at 140.2 99.2) (size 0.8) (drill 0.4) (layers F.Cu B.Cu) (net 2))
   (via (at 138.5 100) (size 0.8) (drill 0.4) (layers F.Cu B.Cu) (net 2))
   (via (at 138.562998 101.202077) (size 0.8) (drill 0.4) (layers F.Cu B.Cu) (net 2))
@@
   (segment (start 147.25 101.2505) (end 147.447 101.4475) (width 0.3) (layer B.Cu) (net 17))
   (segment (start 147.25 101) (end 147.25 101.2505) (width 0.3) (layer B.Cu) (net 17))
+  (segment (start 148.683 99.953) (end 148.73 100) (width 0.3) (layer F.Cu) (net 18))
+  (segment (start 146.1155 99.953) (end 148.683 99.953) (width 0.3) (layer F.Cu) (net 18))
+  (segment (start 142.790332 99.953) (end 142.151332 99.314) (width 0.3) (layer F.Cu) (net 19))
+  (segment (start 143.1905 99.953) (end 142.790332 99.953) (width 0.3) (layer F.Cu) (net 19))
+  (segment (start 142.151332 99.314) (end 142.1384 99.314) (width 0.3) (layer F.Cu) (net 19))
+  (segment (start 142.1384 99.314) (end 141.9352 99.1108) (width 0.3) (layer F.Cu) (net 19))
+  (segment (start 141.584066 98.604569) (end 141.584066 98.708866) (width 0.3) (layer F.Cu) (net 19))
+  (segment (start 142.1384 99.2632) (end 142.1384 99.314) (width 0.3) (layer F.Cu) (net 19))
+  (segment (start 141.584066 98.708866) (end 142.1384 99.2632) (width 0.3) (layer F.Cu) (net 19))
+  (segment (start 143.562569 95.705431) (end 143.588153 95.679847) (width 0.3) (layer F.Cu) (net 21))
+  (segment (start 141.371934 95.705431) (end 143.562569 95.705431) (width 0.3) (layer F.Cu) (net 21))
   (segment (start 145.97 107.53) (end 145.99499 107.50501) (width 0.35) (layer F.Cu) (net 22))
   (segment (start 145.93 107.53) (end 145.97 107.53) (width 0.35) (layer F.Cu) (net 22))
@@
   (segment (start 141.75 101.9885) (end 141.7575 101.981) (width 0.3) (layer B.Cu) (net 22))
   (segment (start 141.75 103.25) (end 141.75 101.9885) (width 0.3) (layer B.Cu) (net 22))
-  (segment (start 148.683 99.953) (end 148.73 100) (width 0.3) (layer F.Cu) (net 18))
-  (segment (start 146.1155 99.953) (end 148.683 99.953) (width 0.3) (layer F.Cu) (net 18))
-  (segment (start 142.790332 99.953) (end 142.151332 99.314) (width 0.3) (layer F.Cu) (net 19))
-  (segment (start 143.1905 99.953) (end 142.790332 99.953) (width 0.3) (layer F.Cu) (net 19))
-  (segment (start 142.151332 99.314) (end 142.1384 99.314) (width 0.3) (layer F.Cu) (net 19))
-  (segment (start 142.1384 99.314) (end 141.9352 99.1108) (width 0.3) (layer F.Cu) (net 19))
-  (segment (start 141.584066 98.604569) (end 141.584066 98.708866) (width 0.3) (layer F.Cu) (net 19))
-  (segment (start 142.1384 99.2632) (end 142.1384 99.314) (width 0.3) (layer F.Cu) (net 19))
-  (segment (start 141.584066 98.708866) (end 142.1384 99.2632) (width 0.3) (layer F.Cu) (net 19))
-  (segment (start 143.562569 95.705431) (end 143.588153 95.679847) (width 0.3) (layer F.Cu) (net 21))
-  (segment (start 141.371934 95.705431) (end 143.562569 95.705431) (width 0.3) (layer F.Cu) (net 21))
   (segment (start 142.195 100.457) (end 141.7575 100.457) (width 0.3) (layer B.Cu) (net 22))
   (segment (start 142.8 99.8) (end 142.195 100.457) (width 0.3) (layer B.Cu) (net 22))

Commit message: minor edits
Other:
- board text added: "1" Fast Detector AW2020-05-12"
- board text removed: "1" Fast Detector AW2020-01-31"
Changed lines of the file:
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@@
-(kicad_pcb (version 20171130) (host pcbnew 5.1.5-52549c5~86~ubuntu19.10.1)
+(kicad_pcb (version 20171130) (host pcbnew 5.1.5-52549c5~86~ubuntu18.04.1)
   (general
     (thickness 1.6)
@@
     (44 Edge.Cuts user)
     (45 Margin user)
-    (46 B.CrtYd user hide)
-    (47 F.CrtYd user hide)
+    (46 B.CrtYd user)
+    (47 F.CrtYd user)
     (48 B.Fab user hide)
     (49 F.Fab user hide)
@@
   (gr_line (start 155 109) (end 155 106.5) (layer B.SilkS) (width 0.12))
   (gr_line (start 145.5 109) (end 155 109) (layer B.SilkS) (width 0.12))
-  (gr_text "1\" Fast Detector\nAW2020-01-31" (at 150.25 107.75) (layer B.SilkS)
+  (gr_text "1\" Fast Detector\nAW2020-05-12" (at 150.25 107.75) (layer B.SilkS)
     (effects (font (size 0.7 0.7) (thickness 0.1)) (justify mirror))
   )
