File: SOT23/circulaire.kicad_pcb (KiCad board)
At the start: 2 copper layers, 25 x 25 mm, 37 parts, among them J101 Conn_Coaxial, J102 Conn_01x03, U101 LT3042xMSE, U102 LT3093xMSE, U103 OPA847xDBV

Commit message: add ohwr-texts
Other:
- board text added: "Copyright Anders E E Wallin, 2020. This documentation describes Open Hardware and is licensed under the CERN OHL v. 1.2. You may redistribute and modify this documentation under the terms of the CERN OHL v.1.2. (http://ohwr.org/cernohl). This documentation is distributed WITHOUT ANY EXPRESS OR IMPLIED WARRANTY, INCLUDING OF MERCHANTABILITY, SATISFACTORY QUALITY AND FITNESS FOR A PARTICULAR PURPOS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"
- board text added: "Thorlabs lens-mount SM1RR clear aperture 22.9mm"
- board text removed: "SM1RR clear aperture 22.9mm"
Changed lines of the file:
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@@
   (general
     (thickness 1.6)
-    (drawings 23)
+    (drawings 28)
     (tracks 294)
     (zones 0)
@@
   )
   (page A4)
+  (title_block
+    (title "1\" Photodetector - SOT23")
+    (date 2020-02)
+    (company "anders.e.e.wallin \"at\" gmail.com")
+  )
   (layers
     (0 F.Cu signal)
@@
     )
   )
+  (gr_line (start 180 50) (end 180 20) (layer Dwgs.User) (width 0.15))
+  (gr_line (start 275 50) (end 180 50) (layer Dwgs.User) (width 0.15))
+  (gr_line (start 275 20) (end 275 50) (layer Dwgs.User) (width 0.15))
+  (gr_line (start 180 20) (end 275 20) (layer Dwgs.User) (width 0.15))
+  (gr_text "Copyright Anders E E Wallin, 2020.\nThis documentation describes Open Hardware and is licensed under the\nCERN OHL v. 1.2.\nYou may redistribute and modify this documentation under the terms of the\nCERN OHL v.1.2. (http://ohwr.org/cernohl). This documentation is distributed\nWITHOUT ANY EXPRESS OR IMPLIED WARRANTY, INCLUDING OF\nMERCHANTABILITY, SATISFACTORY QUALITY AND FITNESS FOR A\nPARTICULAR PURPOSE. Please see the CERN OHL v.1.2 for applicable\nconditions\n" (at 183.4 34.2) (layer Dwgs.User)
+    (effects (font (size 1.5 1.5) (thickness 0.3)) (justify left))
+  )
   (gr_text - (at 160.25 101) (layer F.SilkS)
     (effects (font (size 1 1) (thickness 0.15)))
@@
     (arrow2b (pts (xy 137.5 127.5) (xy 138.626504 126.913579)))
   )
-  (gr_text "SM1RR clear aperture 22.9mm" (at 126.25 78) (layer Dwgs.User)
+  (gr_text "Thorlabs lens-mount\nSM1RR clear aperture 22.9mm" (at 116 73) (layer Dwgs.User)
     (effects (font (size 1 1) (thickness 0.15)))
   )

Commit message: kicad6 version
Parts:
- removed +LED, -LED: LED_ALT, LED_SMD:LED_0805_2012Metric
- removed C110, C111: C, Capacitor_SMD:C_0603_1608Metric
- removed R103, R105, R108: R, Resistor_SMD:R_0603_1608Metric
- C102: value C -> 4u7
- C104: value C -> 10n
- C108, C109: value C -> 100n
- R106: renamed from ROUT; value R -> 49R9
- renumbered CF to C115, PD to D102, +RSET to R101, -RSET to R107, RF to RF101
Connections:
- D102 pad 2: Net-(D102-Pad2) -> GND
- U101 pad 4: Net-(U101-Pad4) -> unconnected-(U101-Pad4)
- U102 pad 4: Net-(U102-Pad4) -> unconnected-(U102-Pad4)
- U102 pad 7: Net-(U102-Pad7) -> unconnected-(U102-Pad7)
- U103 pad 5: Net-(U103-Pad5) -> unconnected-(U103-Pad5)
Routing:
- net Net-(D102-Pad2): track 2.94 -> 0.00 mm
- net GND: track 58.3 -> 60.8 mm
- net Net-(D104-Pad1): track 1.72 -> 0.00 mm
- net Net-(D105-Pad2): track 1.47 -> 0.00 mm
- net /+V: track 24.4 -> 23.1 mm
Other:
- net class Default removed
- net class PWR removed
