File: OPA818/oip_opa818.kicad_pcb (KiCad board)
At the start: 2 copper layers, 25 x 25 mm, 32 parts, among them J101 Conn_Coaxial, J102 Conn_01x03, U101 LT3042xMSE, U102 LT3093xMSE, U103 OPA818IDRGx, U104 BUF602xDBV

Commit message: kicad9 update
Parts:
- U102: footprint Package_SO:MSOP-12-1EP_3x4mm_P0.65mm_EP1.65x2.85mm -> Package_SO:MSOP-12-1EP_3x4.039mm_P0.65mm_EP1.651x2.845mm
- U103: footprint awallinKiCadFootprints:WSON-8-1EP_3x3mm_P0.5mm_EP1.45x2.4mm -> Package_SON:WSON-8-1EP_3x3mm_P0.5mm_EP1.45x2.4mm
Connections:
- R1 pad 1: Net-(R1-Pad1) -> Net-(U103-+)
- U103 pad 3: Net-(R1-Pad1) -> GND
- U103 pad 4: GND -> Net-(U103-+)
