File: OPA818/oip_opa818.kicad_sch (KiCad schematic)
At the start: 32 parts, among them J101 Conn_Coaxial, J102 Conn_01x03, U101 LT3042xMSE, U102 LT3093xMSE, U103 OPA818IDRGx, U104 BUF602xDBV

Commit message: kicad9 update
Parts:
- U102: footprint Package_SO:MSOP-12-1EP_3x4mm_P0.65mm_EP1.65x2.85mm -> Package_SO:MSOP-12-1EP_3x4.039mm_P0.65mm_EP1.651x2.845mm
- U103: footprint awallinKiCadFootprints:WSON-8-1EP_3x3mm_P0.5mm_EP1.45x2.4mm -> Package_SON:WSON-8-1EP_3x3mm_P0.5mm_EP1.45x2.4mm; symbol oip_opa818-rescue:OPA818IDRGx-aw-oip_opa818-rescue-oip_opa818-rescue-oip_opa818-rescue -> Amplifier_Operational:OPA818xDRG
Connections:
- net GND: now also U103.3 (-); no longer U103.4 (+)
- net at R1.1: now also U103.4 (+); no longer U103.3 (-)
